File: RS232_TTL_Converter.kicad_sch (KiCad schematic)
At the start: 19 parts, among them J1 DB9_Female, U1 MAX3232

Commit message: added BOM, need to check PCB thickness
Parts:
- J1: footprint Connector_Dsub:DSUB-9_Female_EdgeMount_P2.77mm -> Connector_Dsub:DSUB-9_Pins_EdgeMount_P2.77mm
